File: devboard.kicad_pcb (KiCad board)
At the start: 2 copper layers, 21 x 51 mm, 50 parts, among them J1 USB_C_Receptacle_USB2.0_14P, J2 Conn_01x20, J3 Conn_01x20, J4 Conn_01x03, J5 Barrel_Jack_Switch, J6 Motor A, J7 Motor B, SW1 SW_Push, U1 RP2040, U2 NCP1117-3.3_SOT223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

Commit message: finished first prototype
Parts:
- removed J4: Conn_01x03, Connector:FanPinHeader_1x03_P2.54mm_Vertical
- removed U2: NCP1117-3.3_SOT223, Package_TO_SOT_SMD:SOT-223-3_TabPin2
- added G***: LOGO, Graphics:medium_statix, B.Cu at (161.0, 67.5)
- C18, C19, C20, C21, C22, C23, C24, C25, D1, D2, L1, U4, U5: moved to B.Cu
- moved C1 140.7 mm to (166.0, 68.0), turned to 45 degrees
- moved C2 140.3 mm to (162.0, 78.8), turned to -90 degrees
- moved R5 139.2 mm to (160.5, 78.5), turned to 180 degrees
- moved C9 138.8 mm to (166.0, 74.0)
- moved R4 138.0 mm to (162.6, 67.0), turned to -90 degrees
- moved R7 137.9 mm to (165.5, 61.0), turned to -90 degrees
- moved R3 137.6 mm to (161.6, 67.0), turned to 90 degrees
- moved C8 137.4 mm to (165.5, 69.5)
- moved C10 137.0 mm to (163.0, 78.8), turned to -90 degrees
- moved C5 136.8 mm to (164.5, 68.0), turned to 90 degrees
- moved R1 135.8 mm to (162.0, 55.0), turned to -90 degrees
- moved C7 133.1 mm to (163.0, 61.5), turned to 90 degrees
- moved C11 133.0 mm to (163.5, 67.5), turned to 90 degrees
- moved C6 132.7 mm to (162.0, 63.5), turned to 90 degrees
- moved R2 131.9 mm to (158.5, 55.0), turned to 90 degrees
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Connections:
- J2 pad 11: STBY -> GPIO8
- U1 pad 11: STBY -> GPIO8
- U1 pad 24: SWCLK -> unconnected-(U1-SWCLK-Pad24)
- U1 pad 25: SWD -> unconnected-(U1-SWDIO-Pad25)
- U4 pad 1: unconnected-(U4-FB-Pad1) -> +3V3_BUCK
- U5 pad 19: STBY -> +3V3
Routing:
- net GND: track 0.00 -> 150.2 mm, vias 0 -> 35
- net +3V3: track 0.00 -> 109.3 mm, vias 0 -> 9
- net /Motor and Power/+12V: track 0.00 -> 80.7 mm, vias 0 -> 1
- net AIN1: track 0.00 -> 29.9 mm, vias 0 -> 2
- net AIN2: track 0.00 -> 29.5 mm, vias 0 -> 1
- net +1V1: track 0.00 -> 27.1 mm, vias 0 -> 2
- net GPIO0: track 0.00 -> 26.4 mm, vias 0 -> 1
- net /Motor and Power/BO1: track 0.00 -> 24.6 mm
- net PWMA: track 0.00 -> 24.4 mm, vias 0 -> 1
- net GPIO15: track 0.00 -> 24.1 mm
- net GPIO1: track 0.00 -> 23.8 mm, vias 0 -> 1
- net GPIO29_ADC3: track 0.00 -> 22.9 mm, vias 0 -> 2
- net GPIO16: track 0.00 -> 22.8 mm
- net QSPI_SS: track 0.00 -> 22.2 mm, vias 0 -> 2
- net BIN2: track 0.00 -> 22.2 mm
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- added copper zone on B.Cu, net GND
- added copper zone on F.Cu, net GND
- added copper zone on In1.Cu, net GND
- added copper zone on In2.Cu, net GND
Other:
- board size 21 x 51 mm -> 21 x 69.8 mm
- copper layers 2 -> 4
- board text added: "2026"
- board text added: "Designed by Satej Gandre"
- board text added: "kineticBoard v0.1"
- board text added: "statixlabs.org"
